File: jafar-se.kicad_sch (KiCad schematic)
At the start: 15 parts, among them J1 XBOX LPC, J2 JTAG, J3 D0 (1.0-1.4), U1 LC4032V-75TN44I, U2 SST49LF080A-33-4C-NHE

Commit message: Finish BOM minus socket
Parts:
- D1: Distributor Link 1 (none) -> https://www.digikey.com/en/products/detail/liteon/LTST-C171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; Distributor Link 2 (none) -> https://www.mouser.com/en/ProductDetail/LITEON/LTST-C171GKT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; LCSC C34499 -> C913075; Manufacturer Hubei KENTO Elec -> Lite-On; Manufacturer Part Number KT-0805W -> LTST-C171GKT
- J1: Distributor Link 1 (none) -> https://www.digikey.com/en/products/detail/te-connectivity-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; Distributor Link 2 (none) -> https://www.mouser.com/en/ProductDetail/TE-Connectivity/5-5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; LCSC (none) -> C18078145; Manufacturer (none) -> Bossie; Manufacturer Part Number (none) -> BX-PM2.54-2-6PY
- J2: now not fitted
- J3: value D0 (1.0-1.4) -> D0; now left out of the parts list
- JP2: value LFRAME (1.6) -> L1
- R1: Distributor Link 1 (none) -> https://www.digikey.com/en/products/detail/yageo/RC0805FR-0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; Distributor Link 2 (none) -> https://www.mouser.com/en/ProductDetail/YAGEO/RC0805FR-071K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; LCSC C2907232 -> C95781; Manufacturer Fojan -> Yageo; Manufacturer Part Number FRC0805F1001TS -> RC0805FR-071KL
