File: jafar-se.kicad_sch (KiCad schematic)
At the start: 15 parts, among them J1 XBOX LPC, J2 JTAG, J3 D0, U1 LC4032V-75TN44I, U2 SST49LF080A-33-4C-NHE

Commit message: Add PLCC-32 socket to schematic so that it shows up in the BOM
Parts:
- added J4: PLCC-32 Socket, Library:PLCC-32_SMD-Socket, symbol Connector:Conn_01x32_Socket
- U2: footprint Library:PLCC-32_SMD-Socket -> Package_LCC:PLCC-32_11.4x14.0mm_P1.27mm
Connections:
- net +3V3: now also J4.10 (Pin_10), J4.11 (Pin_11), J4.12 (Pin_12), J4.24 (Pin_24), J4.25 (Pin_25), J4.3 (Pin_3), J4.30 (Pin_30), J4.32 (Pin_32), J4.4 (Pin_4), J4.5 (Pin_5), J4.6 (Pin_6), J4.7 (Pin_7), J4.8 (Pin_8), J4.9 (Pin_9)
- net FLAD0: now also J4.13 (Pin_13)
- net FLAD1: now also J4.14 (Pin_14)
- net FLAD2: now also J4.15 (Pin_15)
- net FLAD3: now also J4.17 (Pin_17)
- net GND: now also J4.16 (Pin_16), J4.28 (Pin_28), J4.29 (Pin_29)
- net XLCLK: now also J4.31 (Pin_31)
- net ~{FLFRAME}: now also J4.23 (Pin_23)
- net ~{XLRESET}: now also J4.2 (Pin_2)
- no-connect marks 21 -> 29
Other:
- moved on the sheet: C1, C2, C3, C4, C5, C6, D1, R1, U2
