File: jafar-se.kicad_pcb (KiCad board)
At the start: 2 copper layers, 33 x 41 mm, 16 parts, among them J1 XBOX LPC, J2 JTAG, J3 D0, J4 PLCC-32 Socket, U1 LC4032V-75TN44I

Commit message: Cleanup
Routing:
- net +3V3: track 163.2 -> 173.9 mm
- net /~{XLRESET}: track 40.6 -> 40.9 mm, vias 6 -> 4
- net GND: vias 51 -> 67
- net /XLCLK: vias 1 -> 0

Commit message: Cleanup
Parts:
- moved C5 0.89 mm to (131.2, 66.4)
Routing:
- net /FLAD0: track 22.9 -> 34.3 mm, vias 2 -> 0
- net /FLAD1: track 24.4 -> 31.6 mm, vias 2 -> 0
- net /FLAD2: track 24.4 -> 30.0 mm, vias 2 -> 0
- net /FLAD3: track 23.1 -> 26.9 mm, vias 2 -> 0
- net +3V3: track 173.9 -> 170.8 mm
- net /~{XLRESET}: track 40.9 -> 42.7 mm, vias 4 -> 3
- net /~{FLFRAME}: track 16.1 -> 16.7 mm, vias 2 -> 0
- net GND: vias 67 -> 59
- net /XLCLK: vias 0 -> 1

Commit message: Fix DRC
Routing:
- net +3V3: track 170.8 -> 170.3 mm
- net /~{XLRESET}: track 42.7 -> 42.8 mm, vias 3 -> 5
